File: door/pcb/door/motor.sch (KiCad schematic (older format))
At the start: 4 parts, among them J5 Screw_Terminal_01x02, J6 Screw_Terminal_01x02

Commit message: 100uF für Motortreiber geaddet
Parts:
- added C10: 100uF, symbol Device:CP1_Small
Connections:
- net +5V: now also C10.1
- net GND: now also C10.2
Changed lines of the file:
@@
 	1    0    0    -1
 $EndComp
-Wire Wire Line
-	5200 2600 5200 2500
 NoConn ~ 4600 3200
 Wire Wire Line
@@
 Text Label 4000 2900 0    50   ~ 0
 reset
+$Comp
+L Device:CP1_Small C10
+U 1 1 5BF3360F
+P 5550 2550
+F 0 "C10" V 5778 2550 50  0000 C CNN
+F 1 "100uF" V 5687 2550 50  0000 C CNN
+F 2 "" H 5550 2550 50  0001 C CNN
+F 3 "~" H 5550 2550 50  0001 C CNN
+	1    5550 2550
+	0    -1   -1   0
+$EndComp
+Wire Wire Line
+	5200 2500 5200 2550
+Wire Wire Line
+	5200 2550 5450 2550
+Connection ~ 5200 2550
+Wire Wire Line
+	5200 2550 5200 2600
+Wire Wire Line
+	5650 2550 5950 2550
+Wire Wire Line
+	5950 2550 5950 2350
+$Comp
+L power:GND #PWR021
+U 1 1 5BF33CC8
+P 5950 2350
+F 0 "#PWR021" H 5950 2100 50  0001 C CNN
+F 1 "GND" H 5955 2177 50  0000 C CNN
+F 2 "" H 5950 2350 50  0001 C CNN
+F 3 "" H 5950 2350 50  0001 C CNN
+	1    5950 2350
+	-1   0    0    1
+$EndComp
 $EndSCHEMATC

Commit message: layout überarbeitet
Parts:
- C10: footprint (none) -> Capacitor_SMD:CP_Elec_6.3x5.4
Changed lines of the file:
@@
 F 0 "C10" V 5778 2550 50  0000 C CNN
 F 1 "100uF" V 5687 2550 50  0000 C CNN
-F 2 "" H 5550 2550 50  0001 C CNN
+F 2 "Capacitor_SMD:CP_Elec_6.3x5.4" H 5550 2550 50  0001 C CNN
 F 3 "~" H 5550 2550 50  0001 C CNN
 	1    5550 2550

Commit message: recplaced usb micro jack with barrel-jack, reworked pcb layout
Connections:
- net +5V renamed +9V
Changed lines of the file:
@@
-	1    0    0    -1
-$EndComp
-$Comp
-L power:+5V #PWR014
-U 1 1 5BE887A1
-P 5200 2500
-F 0 "#PWR014" H 5200 2350 50  0001 C CNN
-F 1 "+5V" H 5215 2673 50  0000 C CNN
-F 2 "" H 5200 2500 50  0001 C CNN
-F 3 "" H 5200 2500 50  0001 C CNN
-	1    5200 2500
 	1    0    0    -1
 $EndComp
@@
 	-1   0    0    1
 $EndComp
+$Comp
+L power:+9V #PWR0112
+U 1 1 5BFF1E77
+P 5200 2500
+F 0 "#PWR0112" H 5200 2350 50  0001 C CNN
+F 1 "+9V" H 5215 2673 50  0000 C CNN
+F 2 "" H 5200 2500 50  0001 C CNN
+F 3 "" H 5200 2500 50  0001 C CNN
+	1    5200 2500
+	1    0    0    -1
+$EndComp
 $EndSCHEMATC
