File: CAN-Hub/CAN-Hub.kicad_pcb (KiCad board)
At the start: 2 copper layers, 85 x 56 mm, 11 parts, among them J1 DB9_Male_MountingHoles, J2 DB9_Male_MountingHoles, J3 DB9_Male_MountingHoles, J4 DB9_Male_MountingHoles, J5 DB9_Male_MountingHoles, J6 Connector_Screw_Terminal_01x02, J7 Connector_Screw_Terminal_01x02

Commit message: added readme
Routing:
- net /can+: track 180.9 -> 186.9 mm
- net /can-: track 177.0 -> 171.1 mm

Commit message: verical connectors
Parts:
- J1, J2, J3, J4, J5: footprint Connector_Dsub:DSUB-9_Female_Horizontal_P2.77x2.84mm_EdgePinOffset4.94mm_Housed_MountingHolesOffset7.48mm -> Connector_Dsub:DSUB-9_Female_Vertical_P2.77x2.84mm_MountingHoles
- moved J7 80.2 mm to (167.0, 90.0), turned to 90 degrees
- moved J6 80.2 mm to (167.0, 79.0), turned to 90 degrees
- moved J4 23.9 mm to (140.5, 86.0), turned to 270 degrees
- moved J3 23.8 mm to (126.5, 86.0), turned to 270 degrees
- moved J5 23.3 mm to (98.5, 86.0), turned to 270 degrees
- moved J1 15.0 mm to (112.5, 86.0), turned to 270 degrees
- moved J2 13.3 mm to (154.5, 86.0), turned to 270 degrees
Routing:
- net /can+: track 186.9 -> 75.6 mm
- net /can-: track 171.1 -> 73.7 mm
